File: hdmi2c.kicad_sch (KiCad schematic)
At the start: 56 parts, among them J1 USB_C_Receptacle_USB2.0, J7 HDMI1, J8 HDMI2, Q1 Q_NPN_BEC, Q2 Q_NPN_BEC, Q3 BSS138, Q4 BSS138, Q5 BSS138, Q6 BSS138, Q7 BSS83P, Q8 BSS83P, SW1 reset_sw, SW2 SW_Push_shell, SW3 SW_Push_shell, U1 CP2102N-Axx-xQFN24, U3 ESP32-WROOM-32, U4 MIC5205-5.0YM5, U5 MIC5205-5.0YM5, U6 MIC5504-3.3YM5

Commit message: Add project configuration files and initial scripts for HDMI2C development
Parts:
- removed C6: 2.2uF, Capacitor_SMD:C_0603_1608Metric, symbol Device:C_Small
- removed J8: HDMI2, hdmi2c:WURTH_685119134923_HDMI, symbol Connector:HDMI_A
- removed JP2: HDMI2_SH_GND, Jumper:SolderJumper-2_P1.3mm_Open_RoundedPad1.0x1.5mm, symbol Jumper:SolderJumper_2_Bridged
- removed JP7: HDMI2_SCL, Jumper:SolderJumper-2_P1.3mm_Bridged_RoundedPad1.0x1.5mm, symbol Jumper:Jumper_2_Bridged
- removed JP8: HDMI2_SDA, Jumper:SolderJumper-2_P1.3mm_Bridged_RoundedPad1.0x1.5mm, symbol Jumper:Jumper_2_Bridged
- removed Q4, Q6: BSS138, Package_TO_SOT_SMD:SOT-23, symbol Transistor_FET:BSS138
- removed Q8: BSS83P, Package_TO_SOT_SMD:SOT-23, symbol Transistor_FET:BSS83P
- removed R10, R8: 10k, Resistor_SMD:R_0603_1608Metric, symbol Device:R
- removed R12, R14: 2k, Resistor_SMD:R_0603_1608Metric, symbol Device:R
- removed R20: 2.2k, Resistor_SMD:R_0603_1608Metric, symbol Device:R
- removed R21: 3.3k, Resistor_SMD:R_0603_1608Metric, symbol Device:R
- removed U5: MIC5205-5.0YM5, Package_TO_SOT_SMD:SOT-23-5, symbol Regulator_Linear:MIC5205-5.0YM5
Connections:
- net HDMI2_5V_EN: no longer names the net of U3.31 (IO19)
- net HDMI2_HPD_3.3: no longer names the net of U3.28 (IO17)
- net I2C2_SCL: no longer names the net of U3.8 (IO32)
- net I2C2_SDA: no longer names the net of U3.9 (IO33)
- no-connect marks 49 -> 43

Commit message: Add rev2 prototype files and update design parameters for HDMI2C carrier
Parts:
- removed C1: 2.2uF, Capacitor_SMD:C_0603_1608Metric, symbol Device:C_Small
- removed C2, C3, C5: 1uF, Capacitor_SMD:C_0603_1608Metric, symbol Device:C_Small
- removed C4: 10uF, Capacitor_SMD:C_0603_1608Metric, symbol Device:C_Small
- removed D1: TX, LED_SMD:LED_0603_1608Metric, symbol Device:LED
- removed D2: RX, LED_SMD:LED_0603_1608Metric, symbol Device:LED
- removed J1: USB_C_Receptacle_USB2.0, Connector_USB:USB_C_Receptacle_GCT_USB4085, symbol Connector:USB_C_Receptacle_USB2.0
- removed JP1: HDMI1_SH_GND, Jumper:SolderJumper-2_P1.3mm_Open_RoundedPad1.0x1.5mm, symbol Jumper:SolderJumper_2_Bridged
- removed JP3: HDMI1_SCL, Jumper:SolderJumper-2_P1.3mm_Bridged_RoundedPad1.0x1.5mm, symbol Jumper:Jumper_2_Bridged
- removed JP4: HDMI1_SDA, Jumper:SolderJumper-2_P1.3mm_Bridged_RoundedPad1.0x1.5mm, symbol Jumper:Jumper_2_Bridged
- removed Q1, Q2: Q_NPN_BEC, Package_TO_SOT_SMD:SOT-23, symbol Device:Q_NPN_BEC
- removed Q3, Q5: BSS138, Package_TO_SOT_SMD:SOT-23, symbol Transistor_FET:BSS138
- removed Q7: BSS83P, Package_TO_SOT_SMD:SOT-23, symbol Transistor_FET:BSS83P
- removed R1, R2, R3, R7, R9: 10k, Resistor_SMD:R_0603_1608Metric, symbol Device:R
- removed R11, R13: 2k, Resistor_SMD:R_0603_1608Metric, symbol Device:R
- removed R15: 1k, Resistor_SMD:R_0603_1608Metric, symbol Device:R
- removed R16, R17: 5.1k, Resistor_SMD:R_0603_1608Metric, symbol Device:R
- removed R18: 2.2k, Resistor_SMD:R_0603_1608Metric, symbol Device:R
- removed R19: 3.3k, Resistor_SMD:R_0603_1608Metric, symbol Device:R
- removed R22: 22k, Resistor_SMD:R_0603_1608Metric, symbol Device:R
- removed R23: 47k, Resistor_SMD:R_0603_1608Metric, symbol Device:R
- removed R4: 100k, Resistor_SMD:R_0603_1608Metric, symbol Device:R
- removed R5, R6: 68R, Resistor_SMD:R_0603_1608Metric, symbol Device:R
- removed SW1: reset_sw, Button_Switch_SMD:SW_SPST_Omron_B3FS-101xP, symbol hdmi2c:SW_Push_double
- removed SW2, SW3: SW_Push_shell, hdmi2c:SW_TH_Tactile_Omron_B3F-312x, symbol hdmi2c:SW_Push_shell
- removed U1: CP2102N-Axx-xQFN24, Package_DFN_QFN:QFN-24-1EP_4x4mm_P0.5mm_EP2.6x2.6mm, symbol Interface_USB:CP2102N-Axx-xQFN24
- removed U3: ESP32-WROOM-32, RF_Module:ESP32-WROOM-32, symbol RF_Module:ESP32-WROOM-32
- removed U4: MIC5205-5.0YM5, Package_TO_SOT_SMD:SOT-23-5, symbol Regulator_Linear:MIC5205-5.0YM5
- removed U6: MIC5504-3.3YM5, Package_TO_SOT_SMD:SOT-23-5, symbol Regulator_Linear:MIC5504-3.3YM5
- added C1, C2, C3: 100nF, Capacitor_SMD:C_0603_1608Metric, symbol Device:C
- added R24, R25: 100k, Resistor_SMD:R_0603_1608Metric, symbol Device:R
- added R26, R27: 10k, Resistor_SMD:R_0603_1608Metric, symbol Device:R
- added SW2, SW3: B3U-1000P, Button_Switch_SMD:SW_SPST_B3U-1000P, symbol Switch:SW_Push
- added TP1: HDMI_5V, TestPoint:TestPoint_Pad_D1.0mm, symbol Connector:TestPoint
- added TP2: GND, TestPoint:TestPoint_Pad_D1.0mm, symbol Connector:TestPoint
- added TP3: SCL_5V, TestPoint:TestPoint_Pad_D1.0mm, symbol Connector:TestPoint
- added TP4: SDA_5V, TestPoint:TestPoint_Pad_D1.0mm, symbol Connector:TestPoint
- added U3: XIAO ESP32-C6, hdmi2c:XIAO_ESP32C6_Castellated, symbol hdmi2c:XIAO_ESP32C6
- added U4: TPD12S016PWR, Package_SO:TSSOP-24_4.4x7.8mm_P0.65mm, symbol hdmi2c:TPD12S016PW
- J7: MPN (none) -> 685119134923; Manufacturer (none) -> Wurth Elektronik; Specification (none) -> HDMI Type A receptacle; SMT contacts and plated-slot shell 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
Connections:
- net HDMI1_CKS is gone; now on net GND: J7.11 (CKS)
- net HDMI1_D0S is gone; now on net GND: J7.8 (D0S)
- net HDMI1_D1S is gone; now on net GND: J7.5 (D1S)
- net HDMI1_D2S is gone; now on net GND: J7.2 (D2S)
- net +3V3: now also C2.1, R26.1, R27.1, U3.12 (3V3_OUT), U4.24 (VCCA)
- net GND: now also J7.SH, C1.2, C2.2, C3.2, R24.2, R25.2, SW2.2, SW3.2, TP2.1, U3.13 (GND), U4.14 (GND), U4.19 (GND), U4.6 (GND)
- net VBUS: now also C1.1, U3.14 (VBUS / USB 5V), U4.11 (VCC5V)
- net HDMI_HPD_5V: now reaches J7.19 (HPD)
- net HDMI_HPD_5V: now also U4.10 (HPD_B)
- net HDMI1_5V renamed HDMI_5V
- net HDMI_5V: now also C3.1, TP1.1, U4.13 (5V_OUT)
- net HDMI1_CEC: no longer names the net of J7.13 (CEC)
- net HDMI1_SCL renamed HDMI_SCL
- net HDMI_SCL: now also TP3.1, U4.8 (SCL_B)
- net HDMI1_SDA renamed HDMI_SDA
- net HDMI_SDA: now also TP4.1, U4.9 (SDA_B)
- new net BUTTON1: R26.2, SW2.1, U3.9 (D8 / GPIO19)
- new net BUTTON2: R27.2, SW3.1, U3.10 (D9 / GPIO20)
- new net DDC_EN: R25.1, U3.2 (D1 / GPIO1), U4.5 (LS_OE)
- new net HDMI_5V_EN: R24.1, U3.1 (D0 / GPIO0), U4.12 (CT_HPD)
- new net HDMI_HPD: U3.3 (D2 / GPIO2), U4.4 (HPD_A)
- new net I2C_SCL: U3.6 (D5 / GPIO23), U4.2 (SCL_A)
- new net I2C_SDA: U3.5 (D4 / GPIO22), U4.3 (SDA_A)
- no-connect marks 43 -> 24
Other:
- note added: "Enable 5 V before DDC; disable DDC before removing 5 V. Both default off."
- note added: "Firmware: D0=HDMI_5V_EN, D1=DDC_EN, D2=HPD, D4=SDA, D5=SCL."
- note added: "GPIO19/20 buttons are active low. Reserve GPIO3/14 for XIAO RF switch."
- note added: "TMDS and CEC unused; no video passthrough."
- note added: "U3: Seeed XIAO ESP32-C6 V1.0, 14 castellated pads. No battery connection."
- note added: "U4: PW / TSSOP-24 pinout. Integrated pull-ups; no extra DDC pull-ups."
- note added: "USB-powered XIAO carrier / single spare HDMI input"
- note removed: "ESP32"
- note removed: "HDMI"
- note removed: "HDMI 5V"
- note removed: "I2C Level Shifters"
- note removed: "Jumpers & Butts"
- note removed: "Power"
- note removed: "Reset"
- note removed: "Serial Reset/Boot"
- note removed: "USB/Serial"
- company: wlcx industries -> HDMI2C / original project by wlcx
- title: PRJ6 HDMI2C Monitor Controller -> HDMI2C - XIAO ESP32-C6 monitor controller

Commit message: Update creation dates and enhance BOM files for rev2 prototype
Parts:
- C1, C2, C3: LCSC Part # (none) -> C14663; MPN Select to specification -> CC0603KRX7R9BB104; Manufacturer Generic -> YAGEO
- R24, R25: LCSC Part # (none) -> C51048211; MPN Select to specification -> FRH0603B1003TS; Manufacturer Generic -> FOJAN
- R26, R27: LCSC Part # (none) -> C3152123; MPN Select to specification -> SC0603F1002F2BNRH; Manufacturer Generic -> Sunway
- SW2, SW3: LCSC Part # (none) -> C231329
- U3: LCSC Part # (none) -> C27675191; MPN XIAO ESP32-C6 -> 113991254
- U4: LCSC Part # (none) -> C201665
Changed lines of the file:
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@@
 (property "Datasheet" "https://files.seeedstudio.com/wiki/SeeedStudio-XIAO-ESP32C6/XIAO_ESP32_C6_v1.0_SCH_260114.pdf" (at 48.26 57.15 0) (effects (font (size 1.27 1.27)) hide))
 (property "Manufacturer" "Seeed Studio" (at 48.26 57.15 0) (effects (font (size 1.27 1.27)) hide))
-(property "MPN" "XIAO ESP32-C6" (at 48.26 57.15 0) (effects (font (size 1.27 1.27)) hide))
+(property "MPN" "113991254" (at 48.26 57.15 0) (effects (font (size 1.27 1.27)) hide))
+(property "LCSC Part #" "C27675191" (at 48.26 57.15 0) (effects (font (size 1.27 1.27)) hide))
 (property "Specification" "Complete V1.0 module; 14 soldered castellations; 4 MB flash" (at 48.26 57.15 0) (effects (font (size 1.27 1.27)) hide))
 (pin "1")
@@
 (property "Manufacturer" "Texas Instruments" (at 135.89 67.31 0) (effects (font (size 1.27 1.27)) hide))
 (property "MPN" "TPD12S016PWR" (at 135.89 67.31 0) (effects (font (size 1.27 1.27)) hide))
+(property "LCSC Part #" "C201665" (at 135.89 67.31 0) (effects (font (size 1.27 1.27)) hide))
 (property "Specification" "PW/TSSOP-24; do not substitute the RKT pinout" (at 135.89 67.31 0) (effects (font (size 1.27 1.27)) hide))
 (pin "24")
@@
 (property "Footprint" "Capacitor_SMD:C_0603_1608Metric" (at 109.22 116.84 0) (effects (font (size 1.27 1.27)) hide))
 (property "Datasheet" "" (at 109.22 116.84 0) (effects (font (size 1.27 1.27)) hide))
-(property "Manufacturer" "Generic" (at 101.6 116.84 0) (effects (font (size 1.27 1.27)) hide))
-(property "MPN" "Select to specification" (at 101.6 116.84 0) (effects (font (size 1.27 1.27)) hide))
+(property "Manufacturer" "YAGEO" (at 101.6 116.84 0) (effects (font (size 1.27 1.27)) hide))
+(property "MPN" "CC0603KRX7R9BB104" (at 101.6 116.84 0) (effects (font (size 1.27 1.27)) hide))
+(property "LCSC Part #" "C14663" (at 101.6 116.84 0) (effects (font (size 1.27 1.27)) hide))
 (property "Specification" "100 nF; >=16 V; X7R; +/-10%; 0603" (at 101.6 116.84 0) (effects (font (size 1.27 1.27)) hide))
 (pin "1")
@@
 (property "Footprint" "Capacitor_SMD:C_0603_1608Metric" (at 132.07999999999998 116.84 0) (effects (font (size 1.27 1.27)) hide))
 (property "Datasheet" "" (at 132.07999999999998 116.84 0) (effects (font (size 1.27 1.27)) hide))
-(property "Manufacturer" "Generic" (at 124.46 116.84 0) (effects (font (size 1.27 1.27)) hide))
-(property "MPN" "Select to specification" (at 124.46 116.84 0) (effects (font (size 1.27 1.27)) hide))
+(property "Manufacturer" "YAGEO" (at 124.46 116.84 0) (effects (font (size 1.27 1.27)) hide))
+(property "MPN" "CC0603KRX7R9BB104" (at 124.46 116.84 0) (effects (font (size 1.27 1.27)) hide))
+(property "LCSC Part #" "C14663" (at 124.46 116.84 0) (effects (font (size 1.27 1.27)) hide))
 (property "Specification" "100 nF; >=16 V; X7R; +/-10%; 0603" (at 124.46 116.84 0) (effects (font (size 1.27 1.27)) hide))
 (pin "1")
@@
 (property "Footprint" "Capacitor_SMD:C_0603_1608Metric" (at 154.94 116.84 0) (effects (font (size 1.27 1.27)) hide))
 (property "Datasheet" "" (at 154.94 116.84 0) (effects (font (size 1.27 1.27)) hide))
-(property "Manufacturer" "Generic" (at 147.32 116.84 0) (effects (font (size 1.27 1.27)) hide))
-(property "MPN" "Select to specification" (at 147.32 116.84 0) (effects (font (size 1.27 1.27)) hide))
+(property "Manufacturer" "YAGEO" (at 147.32 116.84 0) (effects (font (size 1.27 1.27)) hide))
+(property "MPN" "CC0603KRX7R9BB104" (at 147.32 116.84 0) (effects (font (size 1.27 1.27)) hide))
+(property "LCSC Part #" "C14663" (at 147.32 116.84 0) (effects (font (size 1.27 1.27)) hide))
 (property "Specification" "100 nF; >=16 V; X7R; +/-10%; 0603" (at 147.32 116.84 0) (effects (font (size 1.27 1.27)) hide))
 (pin "1")
@@
 (property "Footprint" "Resistor_SMD:R_0603_1608Metric" (at 40.64 116.84 0) (effects (font (size 1.27 1.27)) hide))
 (property "Datasheet" "" (at 40.64 116.84 0) (effects (font (size 1.27 1.27)) hide))
-(property "Manufacturer" "Generic" (at 33.02 116.84 0) (effects (font (size 1.27 1.27)) hide))
-(property "MPN" "Select to specification" (at 33.02 116.84 0) (effects (font (size 1.27 1.27)) hide))
+(property "Manufacturer" "FOJAN" (at 33.02 116.84 0) (effects (font (size 1.27 1.27)) hide))
+(property "MPN" "FRH0603B1003TS" (at 33.02 116.84 0) (effects (font (size 1.27 1.27)) hide))
+(property "LCSC Part #" "C51048211" (at 33.02 116.84 0) (effects (font (size 1.27 1.27)) hide))
 (property "Specification" "100 kohm; >=0.1 W; +/-1%; 0603" (at 33.02 116.84 0) (effects (font (size 1.27 1.27)) hide))
 (pin "1")
@@
 (property "Footprint" "Resistor_SMD:R_0603_1608Metric" (at 63.5 116.84 0) (effects (font (size 1.27 1.27)) hide))
 (property "Datasheet" "" (at 63.5 116.84 0) (effects (font (size 1.27 1.27)) hide))
-(property "Manufacturer" "Generic" (at 55.88 116.84 0) (effects (font (size 1.27 1.27)) hide))
-(property "MPN" "Select to specification" (at 55.88 116.84 0) (effects (font (size 1.27 1.27)) hide))
+(property "Manufacturer" "FOJAN" (at 55.88 116.84 0) (effects (font (size 1.27 1.27)) hide))
+(property "MPN" "FRH0603B1003TS" (at 55.88 116.84 0) (effects (font (size 1.27 1.27)) hide))
+(property "LCSC Part #" "C51048211" (at 55.88 116.84 0) (effects (font (size 1.27 1.27)) hide))
 (property "Specification" "100 kohm; >=0.1 W; +/-1%; 0603" (at 55.88 116.84 0) (effects (font (size 1.27 1.27)) hide))
 (pin "1")
@@
 (property "Manufacturer" "Omron" (at 189.23 116.84 0) (effects (font (size 1.27 1.27)) hide))
 (property "MPN" "B3U-1000P" (at 189.23 116.84 0) (effects (font (size 1.27 1.27)) hide))
+(property "LCSC Part #" "C231329" (at 189.23 116.84 0) (effects (font (size 1.27 1.27)) hide))
 (property "Specification" "Top-actuated SPST-NO; no locating boss" (at 189.23 116.84 0) (effects (font (size 1.27 1.27)) hide))
 (pin "1")
@@
 (property "Manufacturer" "Omron" (at 237.49 116.84 0) (effects (font (size 1.27 1.27)) hide))
 (property "MPN" "B3U-1000P" (at 237.49 116.84 0) (effects (font (size 1.27 1.27)) hide))
+(property "LCSC Part #" "C231329" (at 237.49 116.84 0) (effects (font (size 1.27 1.27)) hide))
 (property "Specification" "Top-actuated SPST-NO; no locating boss" (at 237.49 116.84 0) (effects (font (size 1.27 1.27)) hide))
 (pin "1")
@@
 (property "Footprint" "Resistor_SMD:R_0603_1608Metric" (at 182.88 133.35 0) (effects (font (size 1.27 1.27)) hide))
 (property "Datasheet" "" (at 182.88 133.35 0) (effects (font (size 1.27 1.27)) hide))
-(property "Manufacturer" "Generic" (at 175.26 133.35 0) (effects (font (size 1.27 1.27)) hide))
-(property "MPN" "Select to specification" (at 175.26 133.35 0) (effects (font (size 1.27 1.27)) hide))
+(property "Manufacturer" "Sunway" (at 175.26 133.35 0) (effects (font (size 1.27 1.27)) hide))
+(property "MPN" "SC0603F1002F2BNRH" (at 175.26 133.35 0) (effects (font (size 1.27 1.27)) hide))
+(property "LCSC Part #" "C3152123" (at 175.26 133.35 0) (effects (font (size 1.27 1.27)) hide))
 (property "Specification" "10 kohm; >=0.1 W; +/-1%; 0603" (at 175.26 133.35 0) (effects (font (size 1.27 1.27)) hide))
 (pin "1")
@@
 (property "Footprint" "Resistor_SMD:R_0603_1608Metric" (at 232.41 133.35 0) (effects (font (size 1.27 1.27)) hide))
 (property "Datasheet" "" (at 232.41 133.35 0) (effects (font (size 1.27 1.27)) hide))
-(property "Manufacturer" "Generic" (at 224.79 133.35 0) (effects (font (size 1.27 1.27)) hide))
-(property "MPN" "Select to specification" (at 224.79 133.35 0) (effects (font (size 1.27 1.27)) hide))
+(property "Manufacturer" "Sunway" (at 224.79 133.35 0) (effects (font (size 1.27 1.27)) hide))
+(property "MPN" "SC0603F1002F2BNRH" (at 224.79 133.35 0) (effects (font (size 1.27 1.27)) hide))
+(property "LCSC Part #" "C3152123" (at 224.79 133.35 0) (effects (font (size 1.27 1.27)) hide))
 (property "Specification" "10 kohm; >=0.1 W; +/-1%; 0603" (at 224.79 133.35 0) (effects (font (size 1.27 1.27)) hide))
 (pin "1")

Commit message: Update creation dates and LCSC part number for J7 in BOM and related files
Parts:
- J7: LCSC Part # (none) -> C2930961
Changed lines of the file:
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@@
 (property "Manufacturer" "Wurth Elektronik" (at 228.6 66.04 0) (effects (font (size 1.27 1.27)) hide))
 (property "MPN" "685119134923" (at 228.6 66.04 0) (effects (font (size 1.27 1.27)) hide))
+(property "LCSC Part #" "C2930961" (at 228.6 66.04 0) (effects (font (size 1.27 1.27)) hide))
 (property "Specification" "HDMI Type A receptacle; SMT contacts and plated-slot shell tabs" (at 228.6 66.04 0) (effects (font (size 1.27 1.27)) hide))
 (pin "1")
